Commit message: gym-pybullet interactive: MuJoCo-parity pinned plant + fully visible 3 paper tests. (1) keyboard module fix + X/Z/B test keys + IJKL flight (WASD/arrows collide with PyBullet GUI camera). (2) color-coded URDF (red front/blue rear arms, prop disks; physics byte-identical: step/sine benchmarks reproduce identical numbers) + _install_urdf now overwrites stale assets. (3) in-window HUD (mode/test/progress/err/motors) + RGB reference-attitude triad + ORBIT/FOLLOW/TOP/FREE cameras. (4) position PIN like MuJoCo: hover thrust + 1kHz pos/linvel pin, angular preserved -- CRITICAL: PyBullet resetBasePositionAndOrientation silently zeroes base velocities, angular must be read BEFORE and restored AFTER (proven: 3.0 rad/s preserved). (5) pinned plant keeps shortest_path=True (benchmark's False stalls the pinned flip at 141 deg; True completes: peak 180 deg, final err <10 deg). VERIFIED pinned: step 57.4 deg peak, sine 30.5 deg/rms 18 deg, flip full inversion + converge, pos hold <= 4 um

File: sim/gym_pybullet/paper_quad.urdf (robot description, URDF)
Before this commit: robot paper_quad, 6 links, 5 joints
Links:
- link prop0_link: geometry visual box size=0.15 0.018 0.006; visual cylinder length=0.0025 radius=0.05
- link prop1_link: geometry visual box size=0.15 0.018 0.006; visual cylinder length=0.0025 radius=0.05
- link prop2_link: geometry visual box size=0.15 0.018 0.006; visual cylinder length=0.0025 radius=0.05
- link prop3_link: geometry visual box size=0.15 0.018 0.006; visual cylinder length=0.0025 radius=0.05
